Commit message: gripper merged ... not working jet

File: schunk_lwa4p_control/urdf/lwa4p.urdf.xacro (robot description, xacro)
@@ -35,3 +35,7 @@
     <origin xyz="0 0 0.5" rpy="0 0 0" />
   </xacro:schunk_lwa4p>
+  <xacro:include filename="$(find schunk_lwa4p_control)/urdf/wsg_50.urdf.xacro" />
+  <xacro:wsg_50_xacro name="gripper" parent="arm_6_link">
+    <origin xyz="0 0 0.08" rpy="0 0 1.570796" />
+  </xacro:wsg_50_xacro>
 </robot>

Commit message: new moveit config

File: schunk_lwa4p_control/urdf/lwa4p.urdf.xacro (robot description, xacro)
@@ -37,5 +37,5 @@
   <xacro:include filename="$(find schunk_lwa4p_control)/urdf/schunk_wsg_50.urdf.xacro" />
   <xacro:wsg_50_xacro name="gripper" parent="arm_6_link">
-    <origin xyz="0 0 0.08" rpy="0 0 1.570796" />
+    <origin xyz="0 0 0.085" rpy="0 0 1.570796" />
   </xacro:wsg_50_xacro>
 </robot>
