Commit message: robot model with finges

File: schunk_description/urdf/lwa4p/lwa4p.urdf.xacro (robot description, xacro)
@@ -100,6 +100,6 @@
       <calibration rising="${arm_3_ref}"/>
       <dynamics damping="5" />
-      <limit effort="176" velocity="0.785" lower="-2.95" upper="2.95"/>
-      <safety_controller k_position="20" k_velocity="50" soft_lower_limit="${-2.95 + 0.01}" soft_upper_limit="${2.95 - 0.01}" />
+      <limit effort="176" velocity="0.785" lower="-2.714" upper="2.714"/>
+      <safety_controller k_position="20" k_velocity="50" soft_lower_limit="${-2.714 + 0.01}" soft_upper_limit="${2.714 - 0.01}" />
     </joint>
     <link name="${name}_3_link">

File: schunk_lwa4p_control/urdf/lwa4p.urdf.xacro (robot description, xacro)
@@ -35,5 +35,5 @@
     <origin xyz="0 0 0.5" rpy="0 0 0" />
   </xacro:schunk_lwa4p>
-  <xacro:include filename="$(find schunk_lwa4p_control)/urdf/wsg_50.urdf.xacro" />
+  <xacro:include filename="$(find schunk_lwa4p_control)/urdf/schunk_wsg_50.urdf.xacro" />
   <xacro:wsg_50_xacro name="gripper" parent="arm_6_link">
     <origin xyz="0 0 0.08" rpy="0 0 1.570796" />

File: schunk_lwa4p_control/urdf/schunk_wsg_50.urdf.xacro (robot description, xacro)
@@ -74,5 +74,5 @@
           </geometry>
           <material name="black">
-		<color rgba="0 0 0 0"/>
+		<color rgba="0 0 0 1"/>
       	  </material>
       </visual>
@@ -113,5 +113,5 @@
           </geometry>
           <material name="black">
-		<color rgba="0 0 0 0"/>
+		<color rgba="0 0 0 1"/>
       	  </material>
       </visual>
@@ -137,4 +137,5 @@
      <dynamics friction="100" damping="100" />
      <limit effort="100" velocity="100"/>
+     <mimic joint="${name}_base_joint_gripper_left" multiplier="-1" offset ="0" />
   </joint>
   <transmission name="${name}_base_trans_right" type="pr2_mechanism_model/SimpleTransmission">
@@ -155,9 +156,9 @@
           <origin xyz="0.0 0 0" rpy="0 0 0" />
           <geometry>
-             <mesh filename="package://schunk_lwa4p_control/meshes/GUIDE_WSG50_110.stl" scale="0.001 0.001 0.001"/>
-	     <!--box size="0.0175 0.03 0.024"/-->
-          </geometry>
-          <material name="black">
-		<color rgba="0 0 0 0"/>
+             <!--box size="0.0175 0.03 0.024"/-->
+             <mesh filename="package://schunk_lwa4p_control/meshes/GUIDE_WSG50_110.stl" scale="0.001 0.001 0.001"/>
+          </geometry>
+          <material name="black">
+		<color rgba="0 0 0 1"/>
       	  </material>
       </visual>
@@ -198,5 +199,5 @@
           </geometry>
           <material name="black">
-		<color rgba="0 0 0 0"/>
+		<color rgba="0 0 0 1"/>
       	  </material>
       </visual>

Commit message: schunk lwa4p urdf model arm lenght fixed

File: schunk_description/urdf/lwa4p/lwa4p.urdf.xacro (robot description, xacro)
@@ -143,12 +143,12 @@
         <origin xyz="0 0 0" rpy="0 0 0" />
         <geometry>
-          <mesh filename="package://schunk_description/meshes/lwa4p/arm_4_link.stl" />
-        </geometry>
-        <material name="Schunk/LightGrey" />
-      </visual>
-      <collision>
-        <origin xyz="0 0 0" rpy="0 0 0" />
-        <geometry>
-          <mesh filename="package://schunk_description/meshes/lwa4p/arm_4_link.stl" />
+          <mesh filename="package://schunk_description/meshes/lwa4p/arm_4_link.stl" scale="0.84 0.84 0.84" />
+        </geometry>
+        <material name="Schunk/LightGrey" />
+      </visual>
+      <collision>
+        <origin xyz="0 0 0" rpy="0 0 0" />
+        <geometry>
+          <mesh filename="package://schunk_description/meshes/lwa4p/arm_4_link.stl" scale="0.84 0.84 0.84" />
         </geometry>
       </collision>
@@ -156,5 +156,5 @@
     <!-- joint between arm_4_link and arm_5_link -->
     <joint name="${name}_5_joint" type="revolute">
-      <origin xyz="0 0.005263 0.365" rpy="1.5708 0 3.14159" />
+      <origin xyz="0 0.005263 0.3049" rpy="1.5708 0 3.14159" />
       <parent link="${name}_4_link"/>
       <child link="${name}_5_link"/>

Commit message: shoring behaviour added

File: schunk_description/urdf/lwa4p/lwa4p.urdf.xacro (robot description, xacro)
@@ -69,6 +69,6 @@
       <calibration rising="${arm_2_ref}"/>
       <dynamics damping="10" />
-      <limit effort="370" velocity="0.785" lower="-2.95" upper="2.95"/>
-      <safety_controller k_position="20" k_velocity="50" soft_lower_limit="${-2.95 + 0.01}" soft_upper_limit="${2.95 - 0.01}" />
+      <limit effort="370" velocity="0.785" lower="-1.55" upper="1.55"/>
+      <safety_controller k_position="20" k_velocity="50" soft_lower_limit="${-1.55 + 0.01}" soft_upper_limit="${1.55 - 0.01}" />
     </joint>
     <link name="${name}_2_link">

File: schunk_lwa4p_control/urdf/lwa4p.urdf.xacro (robot description, xacro)
@@ -20,5 +20,5 @@
       <origin xyz="0 0 0.25" rpy="0 0 0" />
       <geometry>
-         <cylinder radius="0.1" length="0.5"/>
+         <cylinder radius="0.3" length="0.5"/>
       </geometry>
       <material name="Schunk/DarkGrey" />
@@ -27,5 +27,5 @@
       <origin xyz="0 0 0.25" rpy="0 0 0" />
       <geometry>
-        <cylinder radius="0.1" length="0.5"/>
+        <cylinder radius="0.3" length="0.5"/>
       </geometry>
     </collision>
@@ -39,3 +39,7 @@
     <origin xyz="0 0 0.085" rpy="0 0 1.570796" />
   </xacro:wsg_50_xacro>
+  <xacro:include filename="$(find hector_sensors_description)/urdf/asus_camera.urdf.xacro" />
+  <xacro:asus_camera_model name="asus" parent="gripper_base_link">
+    <origin xyz="-0.02 0.055 0.035" rpy="0 -1.570796 -1.570796" />
+  </xacro:asus_camera_model>
 </robot>
