Commit message: hector_obelix_schunk_description: Temporarily fix flippers

File: hector_obelix_schunk_description/urdf/obelix_ugv_schunk_arm.urdf.xacro (robot description, xacro)
@@ -11,8 +11,8 @@
       <!-- use for 2*2 flippers -->
    <obelix_flipper_macro parent="base_link" name="front" front="1">
-     <origin xyz="${base_size_x*0.5} ${base_size_y*0.5+wheel_offset_y+0.5*wheel_size_y}  0 " rpy="0 0 0"/>
+     <origin xyz="${base_size_x*0.5} ${base_size_y*0.5+wheel_offset_y+0.5*wheel_size_y}  0 " rpy="0 -0.78 0"/>
    </obelix_flipper_macro >
   <obelix_flipper_macro parent="base_link" name="back" front="-1">
-    <origin xyz="${-base_size_x*0.5} ${(base_size_y*0.5+wheel_offset_y+0.5*wheel_size_y)}  0  " rpy="0 0 0"/>
+    <origin xyz="${-base_size_x*0.5} ${(base_size_y*0.5+wheel_offset_y+0.5*wheel_size_y)}  0  " rpy="0 0.78 0"/>
   </obelix_flipper_macro >
   <xacro:include filename="$(find schunk_lwa4p)/calibration/calibration.urdf.xacro" />
